File: kicad/scout/scout.kicad_pcb (KiCad board)
At the start: 2 copper layers, 221.4 x 52.3 mm, 96 parts, among them J1 AudioJack2_SwitchT, J2 Conn_01x06_Male, J3 DIN5, J4 DIN5, SW1 SPST, SW10 SPST, SW11 SPST, SW12 SPST, SW13 SPST, SW14 SPST, SW15 SPST, SW16 SPST, SW17 SPST, SW18 SPST, SW19 SPST, SW2 SPST, SW20 SPST, SW21 SPST, SW22 SPST, SW23 SPST, SW24 SPST, SW25 SPST, SW26 SW_SPST, SW3 SPST, SW4 SPST, SW5 SPST, SW6 SPST, SW7 SPST, SW8 SPST, SW9 SPST, U1 ATmega328P-PU, U2 LM386, U3 6N138, Y1 16.00MHz

Commit message: Try to reduce noise and other refinements
* Add decoupling cap before amp
* Add snubber circuit after amp
* Consider bass boost for next rev
* Self-document pin connection assignments in schematic
* Move branding text beyond key area
* Reverse power switch direction
* Enlarge UART hookup labels
Parts:
- removed the Ref** at (226.1, 87.5)
- added C7: .1uF, kicad-official/Capacitor_THT.pretty:C_Disc_D5.0mm_W2.5mm_P5.00mm, F.Cu at (196.0, 84.3)
- added C9: .05uF, kicad-official/Capacitor_THT.pretty:C_Disc_D5.0mm_W2.5mm_P5.00mm, F.Cu at (207.7, 84.3)
- added R14: 10, kicad-official/Resistor_THT.pretty:R_Axial_DIN0207_L6.3mm_D2.5mm_P10.16mm_Horizontal, F.Cu at (205.2, 80.8)
- D1, D10, D11, D12, D13, D14, D15, D16, D17, D18, D19, D2, D20, D21, D22, D23, D24, D25, D3, D4, D5, D6, D7, D8, D9: value D -> 1N4148
- moved Ref** 5.79 mm to (233.6, 82.8)
- moved SW26 4.00 mm to (35.9, 71.7), turned to -90 degrees
Connections:
- net A0 renamed KEYS_R3
- net A1 renamed KEYS_R4
- net A2 renamed KEYS_R5
- net A3 renamed RGB_R
- net A4 renamed POT_1
- net A5 renamed POT_2
- net D10 renamed OSCS_2
- net D11 renamed OSCS_3
- net D12 renamed OSCS_4
- net D13 renamed RGB_B
- net D2 renamed KEYS_C1
- net D3 renamed KEYS_C2
- net D4 renamed KEYS_C3
- net D5 renamed KEYS_D4
- net D6 renamed KEYS_D5
- net D7 renamed KEYS_R1
- net D8 renamed KEYS_R2
- net D9 renamed OSCS_1
- R4 pad 2: Net-(R4-Pad2) -> Net-(C7-Pad1)
- R5 pad 2: Net-(R4-Pad2) -> Net-(C7-Pad1)
- R6 pad 2: Net-(R4-Pad2) -> Net-(C7-Pad1)
- R7 pad 2: Net-(R4-Pad2) -> Net-(C7-Pad1)
- RV1 pad 1: Net-(R4-Pad2) -> Net-(C7-Pad2)
Routing:
- net Net-(R4-Pad2): track 82.2 -> 0.00 mm
- net Net-(C7-Pad1): track 0.00 -> 77.3 mm
- net Net-(C6-Pad1): track 23.1 -> 52.2 mm
- net Net-(C7-Pad2): track 0.00 -> 4.80 mm
- net Net-(C9-Pad2): track 0.00 -> 4.62 mm
- net Net-(C6-Pad2): track 23.2 -> 26.0 mm
Other:
- board text added: "SCOUT2 / PROOF B"
- board text removed: "SCOUT2 / PROOF A"
